Commit message: Stand up first runnable Isaac Lab foosball sim
Replaces the Isaac Gym scaffolding with a DirectRLEnv that loads the
foosball table as an articulation, drops a primitive-sphere ball, and
exposes a standalone viewer runner. Reward and observations are stub —
this iteration is for verifying physics, not training.

Workarounds for Isaac Sim 5.1 URDF importer bugs (digit-prefixed
names, rod-bar OBJ "Used null prim" failure) live in CLAUDE.md; the
upshot is rods import as cylinder primitives and the player meshes
attach as pre-converted USD child prims at scene-setup time.

Adopts src/ layout + UV via pyproject.toml; drops setup.py and the
broken conda bootstrap script.

File: assets/foosball_table/foosball_table.urdf (robot description, URDF)
Before this commit: robot foosball_table, 17 links, 16 joints
Links:
- removed link 2_bar_team_1
- removed link 2_bar_team_2
- removed link 3_bar_team_1
- removed link 3_bar_team_2
- removed link 5_bar_team_1
- removed link 5_bar_team_2
- removed link empty_2_bar_team_1
- removed link empty_2_bar_team_2
- removed link empty_3_bar_team_1
- removed link empty_3_bar_team_2
- removed link empty_5_bar_team_1
- removed link empty_5_bar_team_2
- added link bar2_team_1, mass 0.7638; collision cylinder length=1.08 radius=0.008; visual cylinder length=1.08 radius=0.008
- added link bar2_team_2, mass 0.7638; collision cylinder length=1.08 radius=0.008; visual cylinder length=1.08 radius=0.008
- added link bar3_team_1, mass 0.7638; collision cylinder length=1.08 radius=0.008; visual cylinder length=1.08 radius=0.008
- added link bar3_team_2, mass 0.7638; collision cylinder length=1.08 radius=0.008; visual cylinder length=1.08 radius=0.008
- added link bar5_team_1, mass 0.7638; collision cylinder length=1.08 radius=0.008; visual cylinder length=1.08 radius=0.008
- added link bar5_team_2, mass 0.7638; collision cylinder length=1.08 radius=0.008; visual cylinder length=1.08 radius=0.008
- added link empty_bar2_team_1, mass 0.001; collision box size=0.0005 0.0005 0.0005; visual box size=0.0005 0.0005 0.0005
- added link empty_bar2_team_2, mass 0.001; collision box size=0.0005 0.0005 0.0005; visual box size=0.0005 0.0005 0.0005
- added link empty_bar3_team_1, mass 0.001; collision box size=0.0005 0.0005 0.0005; visual box size=0.0005 0.0005 0.0005
- added link empty_bar3_team_2, mass 0.001; collision box size=0.0005 0.0005 0.0005; visual box size=0.0005 0.0005 0.0005
- added link empty_bar5_team_1, mass 0.001; collision box size=0.0005 0.0005 0.0005; visual box size=0.0005 0.0005 0.0005
- added link empty_bar5_team_2, mass 0.001; collision box size=0.0005 0.0005 0.0005; visual box size=0.0005 0.0005 0.0005
- link empty_goalie_team_1: mass None -> 0.001; geometry collision box size=0.0005 0.0005 0.0005; visual box size=0.0005 0.0005 0.0005
- link empty_goalie_team_2: mass None -> 0.001; geometry collision box size=0.0005 0.0005 0.0005; visual box size=0.0005 0.0005 0.0005
- link goalie_team_1: geometry collision cylinder length=1.08 radius=0.008; visual cylinder length=1.08 radius=0.008
- link goalie_team_2: geometry collision cylinder length=1.08 radius=0.008; visual cylinder length=1.08 radius=0.008
Joints:
- removed joint 2_bar_team_1_prismatic_joint
- removed joint 2_bar_team_1_revolute_joint
- removed joint 2_bar_team_2_prismatic_joint
- removed joint 2_bar_team_2_revolute_joint
- removed joint 3_bar_team_1_prismatic_joint
- removed joint 3_bar_team_1_revolute_joint
- removed joint 3_bar_team_2_prismatic_joint
- removed joint 3_bar_team_2_revolute_joint
- removed joint 5_bar_team_1_prismatic_joint
- removed joint 5_bar_team_1_revolute_joint
- removed joint 5_bar_team_2_prismatic_joint
- removed joint 5_bar_team_2_revolute_joint
- added joint bar2_team_1_prismatic_joint: type prismatic, parent table, child empty_bar2_team_1, origin xyz=0.375 0.0 0.360054, axis 0 1 0, limit lower=-0.187 upper=0.187 effort=9999 velocity=9999
- added joint bar2_team_1_revolute_joint: type revolute, parent empty_bar2_team_1, child bar2_team_1, origin xyz=0 0 0 rpy=0 0 0, axis 0 1 0, limit lower=-100.0 upper=100.0 effort=9999 velocity=9999
- added joint bar2_team_2_prismatic_joint: type prismatic, parent table, child empty_bar2_team_2, origin xyz=-0.375 0.0 0.360054 rpy=0 0 3.1415, axis 0 1 0, limit lower=-0.187 upper=0.187 effort=9999 velocity=9999
- added joint bar2_team_2_revolute_joint: type revolute, parent empty_bar2_team_2, child bar2_team_2, origin xyz=0 0 0 rpy=0 0 0, axis 0 1 0, limit lower=-100.0 upper=100.0 effort=9999 velocity=9999
- added joint bar3_team_1_prismatic_joint: type prismatic, parent table, child empty_bar3_team_1, origin xyz=-0.225 0.0 0.360054, axis 0 1 0, limit lower=-0.117 upper=0.117 effort=9999 velocity=9999
- added joint bar3_team_1_revolute_joint: type revolute, parent empty_bar3_team_1, child bar3_team_1, origin xyz=0 0 0 rpy=0 0 0, axis 0 1 0, limit lower=-100.0 upper=100.0 effort=9999 velocity=9999
- added joint bar3_team_2_prismatic_joint: type prismatic, parent table, child empty_bar3_team_2, origin xyz=0.225 0.0 0.360054 rpy=0 0 3.1415, axis 0 1 0, limit lower=-0.117 upper=0.117 effort=9999 velocity=9999
- added joint bar3_team_2_revolute_joint: type revolute, parent empty_bar3_team_2, child bar3_team_2, origin xyz=0 0 0 rpy=0 0 0, axis 0 1 0, limit lower=-100.0 upper=100.0 effort=9999 velocity=9999
- added joint bar5_team_1_prismatic_joint: type prismatic, parent table, child empty_bar5_team_1, origin xyz=0.075 0.031126 0.360054, axis 0 1 0, limit lower=-0.077 upper=0.077 effort=9999 velocity=9999
- added joint bar5_team_1_revolute_joint: type revolute, parent empty_bar5_team_1, child bar5_team_1, origin xyz=0 0 0 rpy=0 0 0, axis 0 1 0, limit lower=-100.0 upper=100.0 effort=9999 velocity=9999
- added joint bar5_team_2_prismatic_joint: type prismatic, parent table, child empty_bar5_team_2, origin xyz=-0.075 -0.031126 0.360054 rpy=0 0 3.1415, axis 0 1 0, limit lower=-0.077 upper=0.077 effort=9999 velocity=9999
- added joint bar5_team_2_revolute_joint: type revolute, parent empty_bar5_team_2, child bar5_team_2, origin xyz=0 0 0 rpy=0 0 0, axis 0 1 0, limit lower=-100.0 upper=100.0 effort=9999 velocity=9999
- joint goalie_team_1_revolute_joint: limit (none) -> lower=-100.0 upper=100.0 effort=9999 velocity=9999; origin (none) -> xyz=0 0 0 rpy=0 0 0
- joint goalie_team_2_revolute_joint: limit (none) -> lower=-100.0 upper=100.0 effort=9999 velocity=9999; origin (none) -> xyz=0 0 0 rpy=0 0 0
