Commit message: Working physics, single-agent goal scoring, video polish
Physics/geometry fixes so the ball actually plays foosball:
- Field surface at z=0.762, wall top at z=0.912 (matches visible mesh top);
  goal opening z=0.762..0.842 with a 0.07 m cap above.
- Side walls capped at z=0.825, BELOW the rod centerline (z=0.842). Prior
  full-height side walls collided with the rod cylinders and froze the
  prismatic joints — this was the bug behind every earlier "policy only
  spins rods" symptom.
- Goal-mouth roofs above each opening so the ball can't fly out the top.
- URDF: replaced degenerate iyy=0 rod inertias with 0.0001, patched
  empty-link inertials, dropped self-closing link placeholders that were
  crashing the URDF importer.

Reward for single-policy "score any goal":
- Big terminal goal bonus (+100, either net), mild OOB penalty (-10),
  small step penalty (-0.01) for time pressure.
- Potential-based v_toward_goal shaping signed by sign(bx) so the ball
  moving toward whichever net is closer earns +reward; oscillating nets
  zero (episode-sum telescopes to |x_final| - |x_initial|).

Env conveniences:
- Ball color changed to bright orange (contrast against wood + rods).
- LPF disabled by default (alpha=1.0); the ~50 ms filter that shipped
  before muted rod swings so much the policy couldn't actually kick.
- Per-team goal classifier + score counters kept and logged
  (score/team1_total, score/team2_total in TensorBoard).
- Optional random initial ball velocity + curriculum-decayed spawn
  (both no-ops at defaults; opt-in for reward-shaping experiments).
- 9 primitive cuboid colliders (floor + 2 side walls + 4 back-wall
  segments flanking each goal + 2 goal-mouth roofs). Toggleable green
  translucent visualization via visualize_primitive_collision.

Scripts:
- play_foos.py: --spawn_cycle for 5-position ball-drop demo,
  --show_colliders to overlay the primitive walls, --video with
  --video_warmup to skip the initial dark frames.
- replay_foos.py: --spawn_x_near/_far/_vx overrides and --no_curriculum
  for evaluating at harder-than-training distributions; same video-warmup.
- train_foos.py: --save_frequency CLI flag; --seed -1 → random.
- build_table_collision.py: offline OBJ→USD collision-mesh baker
  (experimental fallback; still using per-prim cuboids in-runtime).
- rl_games_ppo_cfg.yaml: entropy_coef=0.0001 (kept sigma stable in the
  keep-ball-moving runs).

File: assets/foosball_table/foosball_table.urdf (robot description, URDF)
Before this commit: robot foosball_table, 17 links, 16 joints
Links:
- link empty_bar2_team_1: geometry visual box size=0.0005 0.0005 0.0005
- link empty_bar2_team_2: geometry visual box size=0.0005 0.0005 0.0005
- link empty_bar3_team_1: geometry visual box size=0.0005 0.0005 0.0005
- link empty_bar3_team_2: geometry visual box size=0.0005 0.0005 0.0005
- link empty_bar5_team_1: geometry visual box size=0.0005 0.0005 0.0005
- link empty_bar5_team_2: geometry visual box size=0.0005 0.0005 0.0005
- link empty_goalie_team_1: geometry visual box size=0.0005 0.0005 0.0005
- link empty_goalie_team_2: geometry visual box size=0.0005 0.0005 0.0005
- link table: geometry visual mesh filename=meshes/table.obj scale=0.001 0.001 0.001
